Commit message: Sequence for the ARM with IK.(Only totem now)

File: indomptable/indomptable_model/urdf/indomptable.urdf.xacro (robot description, xacro)
@@ -236,4 +236,10 @@
                         <xacro:bracket_color />
                 </xacro:my_box>
+                <xacro:my_box name="${side}_wrist_roll_link" lwh="0.03 0.05 0.03" xyz="0 0.015 0" rpy="0 0 0" mass="0.055" material="Gazebo/FlatBlack">
+                        <xacro:ax12_color />
+                </xacro:my_box>
+                <xacro:my_box name="${side}_hand_link" lwh="0.05 0.03 0.03" xyz="0 0 0" rpy="0 0 0" mass="0.055" material="Gazebo/FlatBlack">
+                        <xacro:ax12_color />
+                </xacro:my_box>
 <!--
 		<xacro:my_box name="${side}_shoulder_link" lwh="0.025 0.04 0.05" xyz="0 ${reflect*0.02} 0" rpy="0 0 0" mass="0.05" material="Gazebo/WhiteEmissive">
@@ -388,4 +394,18 @@
         <dynamics damping="0.0"/>
         </joint>
+        <joint name="left_wrist_roll_joint" type="fixed">
+        <parent link="left_wrist_link" />
+        <child link="left_wrist_roll_link" />
+        <origin xyz="0.041 0 0" rpy="0 0 0" />
+        <axis xyz="0 1 0" />
+        </joint>
+        <joint name="left_hand_joint" type="revolute">
+        <parent link="left_wrist_roll_link" />
+        <child link="left_hand_link" />
+        <origin xyz="0.042 0 0" rpy="0 0 0" />
+        <limit lower="-2.53" upper="2.53" effort="10" velocity="3" />
+        <axis xyz="1 0 0" />
+        <dynamics damping="0.0"/>
+        </joint>
 <!--
  	<joint name="left_shoulder_joint" type="fixed">

File: indomptable/indomptable_model/urdf/tmp.urdf (robot description, URDF)
Before this commit: robot indomptable, 17 links, 16 joints
Links:
- added link left_hand_link, mass 0.055; collision box size=0.05 0.03 0.03; visual box size=0.05 0.03 0.03
- added link left_wrist_roll_link, mass 0.055; collision box size=0.03 0.05 0.03; visual box size=0.03 0.05 0.03
Joints:
- added joint left_hand_joint: type revolute, parent left_wrist_roll_link, child left_hand_link, origin xyz=0.042 0 0 rpy=0 0 0, axis 1 0 0, limit lower=-2.53 upper=2.53 effort=10 velocity=3
- added joint left_wrist_roll_joint: type fixed, parent left_wrist_link, child left_wrist_roll_link, origin xyz=0.041 0 0 rpy=0 0 0, axis 0 1 0

Commit message: Add slope control for the arm.

File: indomptable/indomptable_model/urdf/indomptable.urdf.xacro (robot description, xacro)
@@ -344,5 +344,5 @@
         <axis xyz="1 0 0" />
         </joint>
-        <joint name="left_soulder_roll_joint" type="revolute">
+        <joint name="left_shoulder_roll_joint" type="revolute">
         <parent link="left_shoulder_roll_link" />
         <child link="left_shoulder_link" />
@@ -358,5 +358,5 @@
         <axis xyz="1 0 0" />
         </joint>
-        <joint name="left_soulder_lift_joint" type="revolute">
+        <joint name="left_shoulder_lift_joint" type="revolute">
         <parent link="left_shoulder_lift_link" />
         <child link="left_shoulder_link2" />

Commit message: Update robot model.

File: indomptable/indomptable_model/urdf/indomptable.urdf.xacro (robot description, xacro)
@@ -183,5 +183,5 @@
  	<link name="world" />
  	-->
-	<xacro:my_box name="base_link" lwh="0.27 0.31 0.003" xyz="0 0 0" rpy="0 0 0" mass="0.5" material="Gazebo/Grey">
+	<xacro:my_box name="base_link" lwh="0.24 0.32 0.003" xyz="0 0 0" rpy="0 0 0" mass="0.5" material="Gazebo/Grey">
 		<xacro:grey2 />
 	</xacro:my_box>
@@ -192,20 +192,23 @@
 		<xacro:black1 />
 	</xacro:my_cylinder>
-	<xacro:my_box name="netbook_level" lwh="0.27 0.31 0.003" xyz="0 0 0" rpy="0 0 0" mass="0.5" material="Gazebo/Grey">
-                <xacro:grey2 />
-        </xacro:my_box>
-	<xacro:my_box name="right_arm_panel" lwh="0.05 0.002 0.14" xyz="0 0 0" rpy="0 0 0" mass="0.5" material="Gazebo/Grey">
-                <xacro:grey2 />
-        </xacro:my_box>
-        <xacro:my_box name="left_arm_panel" lwh="0.05 0.002 0.14" xyz="0 0 0" rpy="0 0 0" mass="0.5" material="Gazebo/Grey">
-                <xacro:grey2 />
-        </xacro:my_box>
-        <xacro:my_box name="back_arm_panel" lwh="0.002 0.136 0.14" xyz="0 0 0" rpy="0 0 0" mass="0.5" material="Gazebo/Grey">
-                <xacro:grey2 />
-        </xacro:my_box>
-        <xacro:my_box name="right_panel" lwh="0.155 0.002 0.34" xyz="0 0 0" rpy="0 0 0" mass="0.5" material="Gazebo/Grey">
-                <xacro:grey2 />
-        </xacro:my_box>
-        <xacro:my_box name="left_panel" lwh="0.155 0.002 0.34" xyz="0 0 0" rpy="0 0 0" mass="0.5" material="Gazebo/Grey">
+	<xacro:my_box name="first_level" lwh="0.24 0.32 0.002" xyz="0 0 0" rpy="0 0 0" mass="0.5" material="Gazebo/Grey">
+                <xacro:grey2 />
+        </xacro:my_box>
+	<xacro:my_box name="netbook_level" lwh="0.2 0.32 0.002" xyz="0 0 0" rpy="0 0 0" mass="0.5" material="Gazebo/Grey">
+                <xacro:grey2 />
+        </xacro:my_box>
+	<xacro:my_box name="top_level" lwh="0.24 0.32 0.002" xyz="0 0 0" rpy="0 0 0" mass="0.5" material="Gazebo/Grey">
+                <xacro:grey2 />
+        </xacro:my_box>
+	<xacro:my_box name="right_arm_panel" lwh="0.025 0.002 0.06" xyz="0 0 0" rpy="0 0 0" mass="0.5" material="Gazebo/Grey">
+                <xacro:grey2 />
+        </xacro:my_box>
+        <xacro:my_box name="left_arm_panel" lwh="0.025 0.002 0.06" xyz="0 0 0" rpy="0 0 0" mass="0.5" material="Gazebo/Grey">
+                <xacro:grey2 />
+        </xacro:my_box>
+        <xacro:my_box name="right_panel" lwh="0.16 0.002 0.34" xyz="0 0 0" rpy="0 0 0" mass="0.5" material="Gazebo/Grey">
+                <xacro:grey2 />
+        </xacro:my_box>
+        <xacro:my_box name="left_panel" lwh="0.16 0.002 0.34" xyz="0 0 0" rpy="0 0 0" mass="0.5" material="Gazebo/Grey">
                 <xacro:grey2 />
         </xacro:my_box>
@@ -221,5 +224,5 @@
                         <xacro:ax12_color />
                 </xacro:my_box>
-                <xacro:my_box name="${side}_shoulder_link2" lwh="0.038 0.05 0.025" xyz="0.007 0 0" rpy="0 0 0" mass="0.05" material="Gazebo/WhiteEmissive">
+                <xacro:my_box name="${side}_shoulder_link2" lwh="0.054 0.05 0.025" xyz="0.027 0 0" rpy="0 0 0" mass="0.05" material="Gazebo/WhiteEmissive">
                         <xacro:bracket_color />
                 </xacro:my_box>
@@ -227,5 +230,5 @@
                         <xacro:ax12_color />
                 </xacro:my_box>
-                <xacro:my_box name="${side}_elbow_link" lwh="0.038 0.05 0.025" xyz="0.007 0 0" rpy="0 0 0" mass="0.05" material="Gazebo/WhiteEmissive">
+                <xacro:my_box name="${side}_elbow_link" lwh="0.054 0.05 0.025" xyz="0.027 0 0" rpy="0 0 0" mass="0.05" material="Gazebo/WhiteEmissive">
                         <xacro:bracket_color />
                 </xacro:my_box>
@@ -233,12 +236,6 @@
                         <xacro:ax12_color />
                 </xacro:my_box>
-                <xacro:my_box name="${side}_wrist_link" lwh="0.038 0.05 0.025" xyz="0.007 0 0" rpy="0 0 0" mass="0.05" material="Gazebo/WhiteEmissive">
+                <xacro:my_box name="${side}_wrist_link" lwh="0.054 0.05 0.025" xyz="0.027 0 0" rpy="0 0 0" mass="0.05" material="Gazebo/WhiteEmissive">
                         <xacro:bracket_color />
-                </xacro:my_box>
-                <xacro:my_box name="${side}_wrist_roll_link" lwh="0.03 0.05 0.03" xyz="0 0.015 0" rpy="0 0 0" mass="0.055" material="Gazebo/FlatBlack">
-                        <xacro:ax12_color />
-                </xacro:my_box>
-                <xacro:my_box name="${side}_hand_link" lwh="0.05 0.03 0.03" xyz="0 0 0" rpy="0 0 0" mass="0.055" material="Gazebo/FlatBlack">
-                        <xacro:ax12_color />
                 </xacro:my_box>
 <!--
@@ -298,13 +295,23 @@
   	</joint>
   	-->
+	<joint name="first_level_joint" type="fixed">
+    	<parent link="base_link" />
+    	<child link="first_level" />
+    	<origin xyz="0 0 0.1" rpy="0 0 0" />
+	</joint>
 	<joint name="netbook_level_joint" type="fixed">
     	<parent link="base_link" />
     	<child link="netbook_level" />
-    	<origin xyz="0 0 0.253" rpy="0 0 0" />
+    	<origin xyz="-0.02 0 0.21" rpy="0 0 0" />
+	</joint>
+	<joint name="top_level_joint" type="fixed">
+    	<parent link="base_link" />
+    	<child link="top_level" />
+    	<origin xyz="0 0 0.34" rpy="0 0 0" />
 	</joint>
 	<joint name="base_laser_bottom_joint" type="fixed">
     	<parent link="base_link" />
     	<child link="base_laser_bottom" />
-    	<origin xyz="0.11 0 0.022" rpy="0 0 0" />
+    	<origin xyz="0.081 0 0.022" rpy="0 0 0" />
 	</joint>
 	<joint name="base_laser_joint" type="fixed">
@@ -314,17 +321,12 @@
 	</joint>
 	<joint name="left_arm_panel_joint" type="fixed">
-    	<parent link="base_link" />
+    	<parent link="netbook_level" />
     	<child link="left_arm_panel" />
-    	<origin xyz="0.075 0.068 0.0715" rpy="0 0 0" />
+    	<origin xyz="0.065 0.09 0.03" rpy="0 0 0" />
 	</joint>
         <joint name="right_arm_panel_joint" type="fixed">
-        <parent link="base_link" />
+        <parent link="netbook_level" />
         <child link="right_arm_panel" />
-        <origin xyz="0.075 -0.068 0.0715" rpy="0 0 0" />
-        </joint>
-        <joint name="back_arm_panel_joint" type="fixed">
-        <parent link="base_link" />
-        <child link="back_arm_panel" />
-        <origin xyz="0.05 0 0.0715" rpy="0 0 0" />
+        <origin xyz="0.065 -0.09 0.03" rpy="0 0 0" />
         </joint>
         <joint name="left_panel_joint" type="fixed">
@@ -341,5 +343,5 @@
         <parent link="left_arm_panel" />
         <child link="left_shoulder_roll_link" />
-        <origin xyz="0 0.016 0.06" rpy="0 0 0" />
+        <origin xyz="0 -0.016 0.005" rpy="0 0 0" />
         <axis xyz="1 0 0" />
         </joint>
@@ -369,5 +371,5 @@
         <parent link="left_shoulder_link2" />
         <child link="left_elbow_servo_link" />
-        <origin xyz="0.051 0 0" rpy="0 0 0" />
+        <origin xyz="0.08 0 0" rpy="0 0 0" />
         <axis xyz="0 1 0" />
         </joint>
@@ -383,5 +385,5 @@
         <parent link="left_elbow_link" />
         <child link="left_wrist_lift_link" />
-        <origin xyz="0.051 0 0" rpy="0 0 0" />
+        <origin xyz="0.08 0 0" rpy="0 0 0" />
         <axis xyz="0 1 0" />
         </joint>
@@ -392,18 +394,4 @@
         <limit lower="-2.53" upper="2.53" effort="10" velocity="3" />
         <axis xyz="0 1 0" />
-        <dynamics damping="0.0"/>
-        </joint>
-        <joint name="left_wrist_roll_joint" type="fixed">
-        <parent link="left_wrist_link" />
-        <child link="left_wrist_roll_link" />
-        <origin xyz="0.041 0 0" rpy="0 0 0" />
-        <axis xyz="0 1 0" />
-        </joint>
-        <joint name="left_hand_joint" type="revolute">
-        <parent link="left_wrist_roll_link" />
-        <child link="left_hand_link" />
-        <origin xyz="0.042 0 0" rpy="0 0 0" />
-        <limit lower="-2.53" upper="2.53" effort="10" velocity="3" />
-        <axis xyz="1 0 0" />
         <dynamics damping="0.0"/>
         </joint>

Commit message: Add the right ARM.

File: indomptable/indomptable_model/urdf/indomptable.urdf.xacro (robot description, xacro)
@@ -282,7 +282,5 @@
 	</xacro:macro>
 	<xacro:arm side="left" reflect="1" />
-<!--
 	<xacro:arm side="right" reflect="-1" />
-	-->
 	<!-- =================== Joint Definitions ==================== -->
 	<!--
@@ -396,4 +394,60 @@
         <dynamics damping="0.0"/>
         </joint>
+        <joint name="right_shoulder_joint" type="fixed">
+        <parent link="right_arm_panel" />
+        <child link="right_shoulder_roll_link" />
+        <origin xyz="0 0.016 0.005" rpy="0 0 0" />
+        <axis xyz="1 0 0" />
+        </joint>
+        <joint name="right_shoulder_roll_joint" type="revolute">
+        <parent link="right_shoulder_roll_link" />
+        <child link="right_shoulder_link" />
+        <origin xyz="0.01 0 0" rpy="0 0 0" />
+        <limit lower="-2.53" upper="2.53" effort="10" velocity="3" />
+        <axis xyz="0 0 1" />
+        <dynamics damping="0.0"/>
+        </joint>
+        <joint name="right_shoulder_joint2" type="fixed">
+        <parent link="right_shoulder_link" />
+        <child link="right_shoulder_lift_link" />
+        <origin xyz="0.051 0 0" rpy="0 0 0" />
+        <axis xyz="1 0 0" />
+        </joint>
+        <joint name="right_shoulder_lift_joint" type="revolute">
+        <parent link="right_shoulder_lift_link" />
+        <child link="right_shoulder_link2" />
+        <origin xyz="0.01 0 0" rpy="0 0 0" />
+        <limit lower="-2.53" upper="2.53" effort="10" velocity="3" />
+        <axis xyz="0 1 0" />
+        <dynamics damping="0.0"/>
+        </joint>
+        <joint name="right_elbow_servo_joint" type="fixed">
+        <parent link="right_shoulder_link2" />
+        <child link="right_elbow_servo_link" />
+        <origin xyz="0.08 0 0" rpy="0 0 0" />
+        <axis xyz="0 1 0" />
+        </joint>
+        <joint name="right_elbow_joint" type="revolute">
+        <parent link="right_elbow_servo_link" />
+        <child link="right_elbow_link" />
+        <origin xyz="0.01 0 0" rpy="0 0 0" />
+        <limit lower="-2.53" upper="2.53" effort="10" velocity="3" />
+        <axis xyz="0 1 0" />
+        <dynamics damping="0.0"/>
+        </joint>
+        <joint name="right_wrist_lift_joint" type="fixed">
+        <parent link="right_elbow_link" />
+        <child link="right_wrist_lift_link" />
+        <origin xyz="0.08 0 0" rpy="0 0 0" />
+        <axis xyz="0 1 0" />
+        </joint>
+        <joint name="right_wrist_joint" type="revolute">
+        <parent link="right_wrist_lift_link" />
+        <child link="right_wrist_link" />
+        <origin xyz="0.01 0 0" rpy="0 0 0" />
+        <limit lower="-2.53" upper="2.53" effort="10" velocity="3" />
+        <axis xyz="0 1 0" />
+        <dynamics damping="0.0"/>
+        </joint>
 <!--
  	<joint name="left_shoulder_joint" type="fixed">

Commit message: Changes in motion control, fake localization, arm manager.

File: indomptable/indomptable_model/urdf/indomptable.urdf.xacro (robot description, xacro)
@@ -221,5 +221,5 @@
                         <xacro:bracket_color />
                 </xacro:my_box>
-                <xacro:my_box name="${side}_shoulder_lift_link" lwh="0.05 0.03 0.03" xyz="0 0 0" rpy="0 0 0" mass="0.055" material="Gazebo/FlatBlack">
+                <xacro:my_box name="${side}_shoulder_lift_link" lwh="0.05 0.03 0.03" xyz="0.015 0 0" rpy="0 0 0" mass="0.055" material="Gazebo/FlatBlack">
                         <xacro:ax12_color />
                 </xacro:my_box>
@@ -238,4 +238,7 @@
                 <xacro:my_box name="${side}_wrist_link" lwh="0.054 0.05 0.025" xyz="0.027 0 0" rpy="0 0 0" mass="0.05" material="Gazebo/WhiteEmissive">
                         <xacro:bracket_color />
+                </xacro:my_box>
+                <xacro:my_box name="${side}_pump_link" lwh="0.026 0.01 0.01" xyz="0 0 0" rpy="0 0 0" mass="0.05" material="Gazebo/WhiteEmissive">
+                        <xacro:ax12_color />
                 </xacro:my_box>
 <!--
@@ -352,4 +355,19 @@
         <dynamics damping="0.0"/>
         </joint>
+	<joint name="left_shoulder_joint2" type="fixed">
+        <parent link="left_shoulder_link" />
+        <child link="left_shoulder_link2" />
+        <origin xyz="0.03 0 0" rpy="0 0 0" />
+        <axis xyz="1 0 0" />
+        </joint>
+	<joint name="left_shoulder_lift_joint" type="revolute">
+        <parent link="left_shoulder_link2" />
+        <child link="left_shoulder_lift_link" />
+        <origin xyz="0.054 0 0" rpy="0 0 0" />
+        <limit lower="-2.53" upper="2.53" effort="10" velocity="3" />
+        <axis xyz="0 1 0" />
+        <dynamics damping="0.0"/>
+        </joint>
+<!--
         <joint name="left_shoulder_joint2" type="fixed">
         <parent link="left_shoulder_link" />
@@ -366,8 +384,9 @@
         <dynamics damping="0.0"/>
         </joint>
+-->
         <joint name="left_elbow_servo_joint" type="fixed">
-        <parent link="left_shoulder_link2" />
+        <parent link="left_shoulder_lift_link" />
         <child link="left_elbow_servo_link" />
-        <origin xyz="0.08 0 0" rpy="0 0 0" />
+        <origin xyz="0.075 0 0" rpy="0 0 0" />
         <axis xyz="0 1 0" />
         </joint>
@@ -394,4 +413,10 @@
         <dynamics damping="0.0"/>
         </joint>
+        <joint name="left_pump_joint" type="fixed">
+        <parent link="left_wrist_link" />
+        <child link="left_pump_link" />
+        <origin xyz="0.067 0 0" rpy="0 0 0" />
+        <axis xyz="0 1 0" />
+        </joint>
         <joint name="right_shoulder_joint" type="fixed">
         <parent link="right_arm_panel" />
@@ -449,4 +474,10 @@
         <axis xyz="0 1 0" />
         <dynamics damping="0.0"/>
+        </joint>
+        <joint name="right_pump_joint" type="fixed">
+        <parent link="right_wrist_link" />
+        <child link="right_pump_link" />
+        <origin xyz="0.067 0 0" rpy="0 0 0" />
+        <axis xyz="0 1 0" />
         </joint>
 <!--

Commit message: Laser position modification. Robot position initialisation. Motion control changements.

File: indomptable/indomptable_model/urdf/indomptable.urdf.xacro (robot description, xacro)
@@ -314,5 +314,5 @@
     	<parent link="base_link" />
     	<child link="base_laser_bottom" />
-    	<origin xyz="0.081 0 0.022" rpy="0 0 0" />
+    	<origin xyz="0.081 0 0.022" rpy="0 0 -0.02" />
 	</joint>
 	<joint name="base_laser_joint" type="fixed">
