Commit message: Add timer and trajectory wrapper.

File: eurobot2013/eurobot2013_models/urdf/ballista.urdf.xacro (robot description, xacro)
@@ -183,5 +183,5 @@
  	<link name="world" />
  	-->
-	<xacro:my_box name="base_link" lwh="0.24 0.32 0.003" xyz="0 0 0" rpy="0 0 0" mass="0.5" material="Gazebo/Grey">
+	<xacro:my_box name="base_link" lwh="0.24 0.3 0.003" xyz="0 0 0" rpy="0 0 0" mass="0.5" material="Gazebo/Grey">
 		<xacro:grey2 />
 	</xacro:my_box>
@@ -192,11 +192,17 @@
 		<xacro:black1 />
 	</xacro:my_cylinder>
-	<xacro:my_box name="first_level" lwh="0.24 0.32 0.002" xyz="0 0 0" rpy="0 0 0" mass="0.5" material="Gazebo/Grey">
-                <xacro:grey2 />
-        </xacro:my_box>
-	<xacro:my_box name="netbook_level" lwh="0.2 0.32 0.002" xyz="0 0 0" rpy="0 0 0" mass="0.5" material="Gazebo/Grey">
-                <xacro:grey2 />
-        </xacro:my_box>
-	<xacro:my_box name="top_level" lwh="0.24 0.32 0.002" xyz="0 0 0" rpy="0 0 0" mass="0.5" material="Gazebo/Grey">
+	<xacro:my_box name="first_level" lwh="0.24 0.3 0.002" xyz="0 0 0" rpy="0 0 0" mass="0.5" material="Gazebo/Grey">
+                <xacro:grey2 />
+        </xacro:my_box>
+	<xacro:my_box name="second_level" lwh="0.12 0.3 0.002" xyz="0 0 0" rpy="0 0 0" mass="0.5" material="Gazebo/Grey">
+                <xacro:grey2 />
+        </xacro:my_box>
+	<xacro:my_box name="third_level" lwh="0.12 0.3 0.002" xyz="0 0 0" rpy="0 0 0" mass="0.5" material="Gazebo/Grey">
+                <xacro:grey2 />
+        </xacro:my_box>
+	<xacro:my_box name="netbook_level" lwh="0.2 0.3 0.002" xyz="0 0 0" rpy="0 0 0" mass="0.5" material="Gazebo/Grey">
+                <xacro:grey2 />
+        </xacro:my_box>
+	<xacro:my_box name="top_level" lwh="0.24 0.3 0.002" xyz="0 0 0" rpy="0 0 0" mass="0.5" material="Gazebo/Grey">
                 <xacro:grey2 />
         </xacro:my_box>
@@ -215,4 +221,5 @@
  	<!-- ============================   Arms   ============================ -->
 	<xacro:macro name="arm" params="side reflect">
+    <!--
                 <xacro:my_box name="${side}_shoulder_roll_link" lwh="0.05 0.03 0.03" xyz="0 0 0" rpy="0 0 0" mass="0.055" material="Gazebo/FlatBlack">
                         <xacro:ax12_color />
@@ -242,44 +249,4 @@
                         <xacro:ax12_color />
                 </xacro:my_box>
-<!--
-		<xacro:my_box name="${side}_shoulder_link" lwh="0.025 0.04 0.05" xyz="0 ${reflect*0.02} 0" rpy="0 0 0" mass="0.05" material="Gazebo/WhiteEmissive">
-			<xacro:bracket_color />
-		</xacro:my_box>
-		<xacro:my_box name="${side}_shoulder_pan_link" lwh="0.03 0.058 0.03" xyz="0 ${reflect*0.012} 0" rpy="0 0 0" mass="0.055" material="Gazebo/FlatBlack">
-			<xacro:ax12_color />
-		</xacro:my_box>
-		<xacro:my_box name="${side}_shoulder_lift_link" lwh="0.03 0.03 0.052" xyz="0 ${reflect*0.009} -0.018" rpy="0 0 0" mass="0.055" material="Gazebo/FlatBlack">
-			<xacro:ax12_color />
-		</xacro:my_box>
-		<xacro:my_box name="${side}_upper_arm_bracket_link" lwh="0.03 0.03 0.005" xyz="0 0 0" rpy="0 0 0" mass="0.02" material="Gazebo/WhiteEmissive">
-			<xacro:bracket_color />
-		</xacro:my_box>
-		<xacro:my_box name="${side}_arm_roll_link" lwh="0.05 0.03 0.03" xyz="-0.013 ${reflect*0.009} 0" rpy="0 0 0" mass="0.055" material="Gazebo/FlatBlack">
-			<xacro:ax12_color />
-		</xacro:my_box>
-		<xacro:my_box name="${side}_upper_elbow_bracket_link" lwh="0.03 0.022 0.005" xyz="0 0 0" rpy="0 0 0" mass="0.02" material="Gazebo/WhiteEmissive">
-			<xacro:bracket_color />
-		</xacro:my_box>
-		<xacro:my_box name="${side}_elbow_servo_link" lwh="0.03 0.03 0.05" xyz="0 0 0" rpy="0 0 0" mass="0.055" material="Gazebo/FlatBlack">
-			<xacro:ax12_color />
-		</xacro:my_box>
-		<xacro:my_box name="${side}_elbow_link" lwh="0.05 0.025 0.038" xyz="0 0 -0.021" rpy="0 0 0" mass="0.05" material="Gazebo/WhiteEmissive">
-			<xacro:bracket_color />
-		</xacro:my_box>
-		<xacro:my_cylinder name="${side}_lower_arm_link" l="0.092" r="0.006" xyz="0.0015 0 -0.048" rpy="0 0 0" mass="0.2" material="Gazebo/Chrome">
-			<xacro:grey1 />
-		</xacro:my_cylinder>
-		<xacro:my_box name="${side}_wrist_bracket_link" lwh="0.05 0.025 0.038" xyz="0 0 -0.021" rpy="0 0 0" mass="0.02" material="Gazebo/WhiteEmissive">
-			<xacro:bracket_color />
-		</xacro:my_box>
-		<xacro:my_box name="${side}_wrist_link" lwh="0.03 0.03 0.05" xyz="0 0 -0.016" rpy="0 0 0" mass="0.055" material="Gazebo/FlatBlack">
-			<xacro:ax12_color />
-		</xacro:my_box>
-		<xacro:my_box name="${side}_hand_link" lwh="0.03 0.01 0.064" xyz="0 0 -0.032" rpy="0 0 0" mass="0.1" material="Gazebo/WhiteEmissive">
-			<xacro:grey1 />
-		</xacro:my_box>
-		<xacro:my_box name="${side}_finger_link" lwh="0.01 0.01 0.005" xyz="0 0 0" rpy="0 0 0" mass="0.001" material="Gazebo/WhiteEmissive">
-			<xacro:black1 />
-		</xacro:my_box>
 -->
 	</xacro:macro>
@@ -287,17 +254,18 @@
 	<xacro:arm side="right" reflect="-1" />
 	<!-- =================== Joint Definitions ==================== -->
-	<!--
-	<joint name="base_world_link" type="continuous">
-    	<parent link="world"/>
-    	<child link="base_link"/>
-    	<axis xyz="0 0 0"/>
-    	<origin rpy="0 0 0" xyz="0 0 0"/>
-    	<dynamics damping="0.05"/>
-  	</joint>
-  	-->
 	<joint name="first_level_joint" type="fixed">
     	<parent link="base_link" />
     	<child link="first_level" />
-    	<origin xyz="0 0 0.1" rpy="0 0 0" />
+    	<origin xyz="0 0 0.011" rpy="0 0 0" />
+	</joint>
+	<joint name="second_level_joint" type="fixed">
+    	<parent link="first_level" />
+    	<child link="second_level" />
+    	<origin xyz="0.06 0 0.07" rpy="0 0 0" />
+	</joint>
+	<joint name="third_level_joint" type="fixed">
+    	<parent link="first_level" />
+    	<child link="third_level" />
+    	<origin xyz="0.06 0 0.17" rpy="0 0 0" />
 	</joint>
 	<joint name="netbook_level_joint" type="fixed">
@@ -312,7 +280,7 @@
 	</joint>
 	<joint name="base_laser_bottom_joint" type="fixed">
-    	<parent link="base_link" />
+    	<parent link="second_level" />
     	<child link="base_laser_bottom" />
-    	<origin xyz="0.081 0 0.022" rpy="0 0 -0.02" />
+    	<origin xyz="0.03 0 0.022" rpy="0 0 -0.02" />
 	</joint>
 	<joint name="base_laser_joint" type="fixed">
@@ -334,11 +302,12 @@
         <parent link="base_link" />
         <child link="left_panel" />
-        <origin xyz="0 0.155 0.17" rpy="0 0 0" />
+        <origin xyz="0 0.15 0.17" rpy="0 0 0" />
         </joint>
         <joint name="right_panel_joint" type="fixed">
         <parent link="base_link" />
         <child link="right_panel" />
-        <origin xyz="0 -0.155 0.17" rpy="0 0 0" />
-        </joint>
+        <origin xyz="0 -0.15 0.17" rpy="0 0 0" />
+        </joint>
+<!--
         <joint name="left_shoulder_joint" type="fixed">
         <parent link="left_arm_panel" />
@@ -369,20 +338,4 @@
         <dynamics damping="0.0"/>
         </joint>
-<!--
-        <joint name="left_shoulder_joint2" type="fixed">
-        <parent link="left_shoulder_link" />
-        <child link="left_shoulder_lift_link" />
-        <origin xyz="0.051 0 0" rpy="0 0 0" />
-        <axis xyz="1 0 0" />
-        </joint>
-        <joint name="left_shoulder_lift_joint" type="revolute">
-        <parent link="left_shoulder_lift_link" />
-        <child link="left_shoulder_link2" />
-        <origin xyz="0.01 0 0" rpy="0 0 0" />
-        <limit lower="-2.53" upper="2.53" effort="10" velocity="3" />
-        <axis xyz="0 1 0" />
-        <dynamics damping="0.0"/>
-        </joint>
--->
         <joint name="left_elbow_servo_joint" type="fixed">
         <parent link="left_shoulder_lift_link" />
@@ -481,4 +434,5 @@
         <axis xyz="0 1 0" />
         </joint>
+-->
 <!--
  	<joint name="left_shoulder_joint" type="fixed">
