Commit message: Beginning of IK for GROS robot.

File: eurobot2014/eurobot2014_models/urdf/field.urdf.xacro (robot description, xacro)
@@ -179,5 +179,5 @@
 		</gazebo>
     </xacro:macro>
-	<link name="map" />
+	<link name="world" />
         <!-- ============================   Hearts   ============================ -->
     <xacro:my_cylinder name="middle_heart" l="0.03" r="0.15" xyz="0 0 0" rpy="0 0 0" mass="0.1" material="Gazebo/Grey">
@@ -265,115 +265,115 @@
     -->
     <joint name="middle_heart_joint" type="fixed">
-    <parent link="map" />
+    <parent link="world" />
     <child link="middle_heart" />
     <origin xyz="0.0 0.95 0.015" rpy="0 0 0" />
     </joint>
     <joint name="right_heart_joint" type="fixed">
-    <parent link="map" />
+    <parent link="world" />
     <child link="right_heart" />
     <origin xyz="1.5 0.0 0.015" rpy="0 0 0" />
     </joint>
     <joint name="left_heart_joint" type="fixed">
-    <parent link="map" />
+    <parent link="world" />
     <child link="left_heart" />
     <origin xyz="-1.5 0.0 0.015" rpy="0 0 0" />
     </joint>
     <joint name="RB_basket_joint" type="fixed">
-    <parent link="map" />
+    <parent link="world" />
     <child link="RB_basket" />
     <origin xyz="0.750 1.785 0.022" rpy="0 0 0" />
     </joint>
     <joint name="LB_basket_joint" type="fixed">
-    <parent link="map" />
+    <parent link="world" />
     <child link="LB_basket" />
     <origin xyz="-0.750 1.785 0.022" rpy="0 0 0" />
     </joint>
     <joint name="RT_basket_joint" type="fixed">
-    <parent link="map" />
+    <parent link="world" />
     <child link="RT_basket" />
     <origin xyz="0.750 1.935 0.035" rpy="0 0 0" />
     </joint>
     <joint name="LT_basket_joint" type="fixed">
-    <parent link="map" />
+    <parent link="world" />
     <child link="LT_basket" />
     <origin xyz="-0.750 1.935 0.035" rpy="0 0 0" />
     </joint>
     <joint name="tree1_joint" type="fixed">
-    <parent link="map" />
+    <parent link="world" />
     <child link="tree1" />
     <origin xyz="1.5 0.7 0.16" rpy="0 0 0" />
     </joint>
     <joint name="tree1_top_joint" type="fixed">
-    <parent link="map" />
+    <parent link="world" />
     <child link="tree1_top" />
     <origin xyz="1.5 0.7 0.325" rpy="0 0 0" />
     </joint>
     <joint name="tree2_joint" type="fixed">
-    <parent link="map" />
+    <parent link="world" />
     <child link="tree2" />
     <origin xyz="-1.5 0.7 0.16" rpy="0 0 0" />
     </joint>
     <joint name="tree2_top_joint" type="fixed">
-    <parent link="map" />
+    <parent link="world" />
     <child link="tree2_top" />
     <origin xyz="-1.5 0.7 0.325" rpy="0 0 0" />
     </joint>
     <joint name="tree3_joint" type="fixed">
-    <parent link="map" />
+    <parent link="world" />
     <child link="tree3" />
     <origin xyz="0.8 0.0 0.16" rpy="0 0 0" />
     </joint>
     <joint name="tree3_top_joint" type="fixed">
-    <parent link="map" />
+    <parent link="world" />
     <child link="tree3_top" />
     <origin xyz="0.8 0.0 0.325" rpy="0 0 0" />
     </joint>
     <joint name="tree4_joint" type="fixed">
-    <parent link="map" />
+    <parent link="world" />
     <child link="tree4" />
     <origin xyz="-0.8 0.0 0.16" rpy="0 0 0" />
     </joint>
     <joint name="tree4_top_joint" type="fixed">
-    <parent link="map" />
+    <parent link="world" />
     <child link="tree4_top" />
     <origin xyz="-0.8 0.0 0.325" rpy="0 0 0" />
     </joint>
     <joint name="inter1_joint" type="fixed">
-    <parent link="map" />
+    <parent link="world" />
     <child link="inter1" />
     <origin xyz="0.6 0.9 0.005" rpy="0 0 0" />
     </joint>
     <joint name="inter2_joint" type="fixed">
-    <parent link="map" />
+    <parent link="world" />
     <child link="inter2" />
     <origin xyz="-0.6 0.9 0.005" rpy="0 0 0" />
     </joint>
     <joint name="inter3_joint" type="fixed">
-    <parent link="map" />
+    <parent link="world" />
     <child link="inter3" />
     <origin xyz="1.1 0.9 0.005" rpy="0 0 0" />
     </joint>
     <joint name="inter4_joint" type="fixed">
-    <parent link="map" />
+    <parent link="world" />
     <child link="inter4" />
     <origin xyz="-1.1 0.9 0.005" rpy="0 0 0" />
     </joint>
     <joint name="up_joint" type="fixed">
-    <parent link="map" />
+    <parent link="world" />
     <child link="up_link" />
     <origin xyz="0.0 -0.005 0.035" rpy="0 0 0" />
     </joint>
     <joint name="down_joint" type="fixed">
-    <parent link="map" />
+    <parent link="world" />
     <child link="down_link" />
     <origin xyz="0.0 2.005 0.035" rpy="0 0 0" />
     </joint>
     <joint name="left_joint" type="fixed">
-    <parent link="map" />
+    <parent link="world" />
     <child link="left_link" />
     <origin xyz="-1.505 1.0 0.035" rpy="0 0 0" />
     </joint>
     <joint name="right_joint" type="fixed">
-    <parent link="map" />
+    <parent link="world" />
     <child link="right_link" />
     <origin xyz="1.505 1.0 0.035" rpy="0 0 0" />

File: eurobot2014/eurobot2014_models/urdf/test.urdf.xacro (robot description, xacro)
@@ -315,5 +315,5 @@
         <child link="Rlink2" />
         <origin xyz="0.0 0 0" rpy="0 0 0" />
-        <limit lower="-2.53" upper="2.53" effort="10" velocity="3" />
+        <limit lower="-0.53" upper="0.53" effort="10" velocity="3" />
         <axis xyz="0 0 1" />
         <dynamics damping="0.0"/>
@@ -323,5 +323,5 @@
         <child link="Rlink3" />
         <origin xyz="0.0797 0 0" rpy="0 0 0" />
-        <limit lower="-2.53" upper="2.53" effort="10" velocity="3" />
+        <limit lower="-2.53" upper="1.57" effort="10" velocity="3" />
         <axis xyz="0 1 0" />
         <dynamics damping="0.0"/>
@@ -339,5 +339,5 @@
         <child link="Rlink5" />
         <origin xyz="0.026 0 0" rpy="0 0 0" />
-        <limit lower="-2.53" upper="2.53" effort="10" velocity="3" />
+        <limit lower="-1.57" upper="1.57" effort="10" velocity="3" />
         <axis xyz="0 1 0" />
         <dynamics damping="0.0"/>
@@ -347,5 +347,5 @@
         <child link="Rlink6" />
         <origin xyz="0.0675 0 0" rpy="0 0 0" />
-        <limit lower="-2.53" upper="2.53" effort="10" velocity="3" />
+        <limit lower="-1.57" upper="1.57" effort="10" velocity="3" />
         <axis xyz="0 1 0" />
         <dynamics damping="0.0"/>

Commit message: First test with the real arms of GROS robot.

File: eurobot2014/eurobot2014_models/urdf/field.urdf.xacro (robot description, xacro)
@@ -241,4 +241,23 @@
     <xacro:black1 />
     </xacro:my_cylinder>
+    <!-- ============================   Fruits   ============================ -->
+    <xacro:my_cylinder name="fruit1" l="0.044" r="0.012" xyz="0 0 0" rpy="0 0 0" mass="0.1" material="Gazebo/Grey">
+    <xacro:black1 />
+    </xacro:my_cylinder>
+    <xacro:my_cylinder name="fruit2" l="0.044" r="0.012" xyz="0 0 0" rpy="0 0 0" mass="0.1" material="Gazebo/Grey">
+    <xacro:black1 />
+    </xacro:my_cylinder>
+    <xacro:my_cylinder name="fruit3" l="0.044" r="0.012" xyz="0 0 0" rpy="0 0 0" mass="0.1" material="Gazebo/Grey">
+    <xacro:black1 />
+    </xacro:my_cylinder>
+    <xacro:my_cylinder name="fruit4" l="0.044" r="0.012" xyz="0 0 0" rpy="0 0 0" mass="0.1" material="Gazebo/Grey">
+    <xacro:black1 />
+    </xacro:my_cylinder>
+    <xacro:my_cylinder name="fruit5" l="0.044" r="0.012" xyz="0 0 0" rpy="0 0 0" mass="0.1" material="Gazebo/Grey">
+    <xacro:black1 />
+    </xacro:my_cylinder>
+    <xacro:my_cylinder name="fruit6" l="0.044" r="0.012" xyz="0 0 0" rpy="0 0 0" mass="0.1" material="Gazebo/Grey">
+    <xacro:black1 />
+    </xacro:my_cylinder>
     <!-- ============================   Border   ============================ -->
     <xacro:my_box name="up_link" lwh="3.0 0.01 0.07" xyz="0 0 0" rpy="0 0 0" mass="0.5" material="Gazebo/FlatBlack">
@@ -359,4 +378,34 @@
     <origin xyz="-1.1 0.9 0.005" rpy="0 0 0" />
     </joint>
+    <joint name="fruit1_joint" type="fixed">
+    <parent link="world" />
+    <child link="fruit1" />
+    <origin xyz="-1.5 0.580 0.158" rpy="0 0 0" />
+    </joint>
+    <joint name="fruit2_joint" type="fixed">
+    <parent link="world" />
+    <child link="fruit2" />
+    <origin xyz="-1.5 0.820 0.208" rpy="0 0 0" />
+    </joint>
+    <joint name="fruit3_joint" type="fixed">
+    <parent link="world" />
+    <child link="fruit3" />
+    <origin xyz="-1.396 0.640 0.208" rpy="0 0 0" />
+    </joint>
+    <joint name="fruit4_joint" type="fixed">
+    <parent link="world" />
+    <child link="fruit4" />
+    <origin xyz="-1.396 0.760 0.158" rpy="0 0 0" />
+    </joint>
+    <joint name="fruit5_joint" type="fixed">
+    <parent link="world" />
+    <child link="fruit5" />
+    <origin xyz="-1.604 0.640 0.158" rpy="0 0 0" />
+    </joint>
+    <joint name="fruit6_joint" type="fixed">
+    <parent link="world" />
+    <child link="fruit6" />
+    <origin xyz="-1.604 0.760 0.208" rpy="0 0 0" />
+    </joint>
     <joint name="up_joint" type="fixed">
     <parent link="world" />
