Commit message: Compute the IK of an ARM.

File: eurobot2014/eurobot2014_models/urdf/test.urdf.xacro (robot description, xacro)
@@ -295,5 +295,5 @@
         </joint>
  	<!-- =================== RIGHT ARM Definitions ==================== -->
-        <joint name="joint1" type="revolute">
+        <joint name="Rarm1_joint" type="revolute">
         <parent link="link1" />
         <child link="link2" />
@@ -303,5 +303,5 @@
         <dynamics damping="0.0"/>
         </joint>
-        <joint name="joint2" type="revolute">
+        <joint name="Rarm2_joint" type="revolute">
         <parent link="link2" />
         <child link="link3" />
@@ -311,5 +311,5 @@
         <dynamics damping="0.0"/>
         </joint>
-        <joint name="joint3" type="revolute">
+        <joint name="Rarm3_joint" type="revolute">
         <parent link="link3" />
         <child link="link4" />
@@ -319,5 +319,5 @@
         <dynamics damping="0.0"/>
         </joint>
-        <joint name="joint4" type="revolute">
+        <joint name="Rarm4_joint" type="revolute">
         <parent link="link4" />
         <child link="link5" />
@@ -327,5 +327,5 @@
         <dynamics damping="0.0"/>
         </joint>
-        <joint name="joint5" type="revolute">
+        <joint name="Rarm5_joint" type="revolute">
         <parent link="link5" />
         <child link="link6" />

Commit message: Lot of changes and improvement for Eurobot2014.

File: eurobot2014/eurobot2014_models/urdf/test.urdf.xacro (robot description, xacro)
@@ -205,20 +205,20 @@
         </xacro:my_cylinder>
  	<!-- ============================   Arms   ============================ -->
-                <xacro:my_box name="link1" lwh="0.04 0.04 0.04" xyz="-0.02 0 0" rpy="0 0 0" mass="0.055" material="Gazebo/FlatBlack">
-                        <xacro:ax12_color />
-                </xacro:my_box>
-		<xacro:my_box name="link2" lwh="0.0797 0.04 0.04" xyz="0.03985 0 0" rpy="0 0 0" mass="0.055" material="Gazebo/WhiteEmissive">
-                        <xacro:bracket_color />
-                </xacro:my_box>
-                <xacro:my_box name="link3" lwh="0.053 0.04 0.04" xyz="0.0265 0 0" rpy="0 0 0" mass="0.05" material="Gazebo/FlatBlack">
-                        <xacro:ax12_color />
-                </xacro:my_box>
-                <xacro:my_box name="link4" lwh="0.026 0.04 0.04" xyz="0.013 0 0" rpy="0 0 0" mass="0.05" material="Gazebo/WhiteEmissive">
-                        <xacro:bracket_color />
-                </xacro:my_box>
-                <xacro:my_box name="link5" lwh="0.0675 0.04 0.04" xyz="0.03375 0 0" rpy="0 0 0" mass="0.05" material="Gazebo/FlatBlack">
-                        <xacro:ax12_color />
-                </xacro:my_box>
-                <xacro:my_box name="link6" lwh="0.04 0.04 0.04" xyz="0.02 0 0" rpy="0 0 0" mass="0.05" material="Gazebo/WhiteEmissive">
+                <xacro:my_box name="Rlink1" lwh="0.04 0.04 0.04" xyz="-0.02 0 0" rpy="0 0 0" mass="0.055" material="Gazebo/FlatBlack">
+                        <xacro:ax12_color />
+                </xacro:my_box>
+		<xacro:my_box name="Rlink2" lwh="0.0797 0.04 0.04" xyz="0.03985 0 0" rpy="0 0 0" mass="0.055" material="Gazebo/WhiteEmissive">
+                        <xacro:bracket_color />
+                </xacro:my_box>
+                <xacro:my_box name="Rlink3" lwh="0.053 0.04 0.04" xyz="0.0265 0 0" rpy="0 0 0" mass="0.05" material="Gazebo/FlatBlack">
+                        <xacro:ax12_color />
+                </xacro:my_box>
+                <xacro:my_box name="Rlink4" lwh="0.026 0.04 0.04" xyz="0.013 0 0" rpy="0 0 0" mass="0.05" material="Gazebo/WhiteEmissive">
+                        <xacro:bracket_color />
+                </xacro:my_box>
+                <xacro:my_box name="Rlink5" lwh="0.0675 0.04 0.04" xyz="0.03375 0 0" rpy="0 0 0" mass="0.05" material="Gazebo/FlatBlack">
+                        <xacro:ax12_color />
+                </xacro:my_box>
+                <xacro:my_box name="Rlink6" lwh="0.04 0.04 0.04" xyz="0.02 0 0" rpy="0 0 0" mass="0.05" material="Gazebo/WhiteEmissive">
                         <xacro:bracket_color />
                 </xacro:my_box>
@@ -226,14 +226,14 @@
                         <xacro:ax12_color />
                 </xacro:my_box>
-                <xacro:my_box name="Llink2" lwh="0.052 0.04 0.04" xyz="0.026 0 0" rpy="0 0 0" mass="0.055" material="Gazebo/WhiteEmissive">
-                        <xacro:bracket_color />
-                </xacro:my_box>
-                <xacro:my_box name="Llink3" lwh="0.0815 0.04 0.04" xyz="0.04075 0 0" rpy="0 0 0" mass="0.05" material="Gazebo/FlatBlack">
-                        <xacro:ax12_color />
-                </xacro:my_box>
-                <xacro:my_box name="Llink4" lwh="0.0415 0.04 0.04" xyz="0.02075 0 0" rpy="0 0 0" mass="0.05" material="Gazebo/WhiteEmissive">
-                        <xacro:bracket_color />
-                </xacro:my_box>
-                <xacro:my_box name="Llink5" lwh="0.052 0.04 0.04" xyz="0.026 0 0" rpy="0 0 0" mass="0.05" material="Gazebo/FlatBlack">
+                <xacro:my_box name="Llink2" lwh="0.0797 0.04 0.04" xyz="0.03985 0 0" rpy="0 0 0" mass="0.055" material="Gazebo/WhiteEmissive">
+                        <xacro:bracket_color />
+                </xacro:my_box>
+                <xacro:my_box name="Llink3" lwh="0.053 0.04 0.04" xyz="0.0265 0 0" rpy="0 0 0" mass="0.05" material="Gazebo/FlatBlack">
+                        <xacro:ax12_color />
+                </xacro:my_box>
+                <xacro:my_box name="Llink4" lwh="0.026 0.04 0.04" xyz="0.013 0 0" rpy="0 0 0" mass="0.05" material="Gazebo/WhiteEmissive">
+                        <xacro:bracket_color />
+                </xacro:my_box>
+                <xacro:my_box name="Llink5" lwh="0.0675 0.04 0.04" xyz="0.03375 0 0" rpy="0 0 0" mass="0.05" material="Gazebo/FlatBlack">
                         <xacro:ax12_color />
                 </xacro:my_box>
@@ -258,5 +258,5 @@
         <joint name="rightarm_joint" type="fixed">
         <parent link="arm_level_link" />
-        <child link="link1" />
+        <child link="Rlink1" />
         <origin xyz="0.05 -0.06 0.032" rpy="0 0 0" />
         </joint>
@@ -296,6 +296,6 @@
  	<!-- =================== RIGHT ARM Definitions ==================== -->
         <joint name="Rarm1_joint" type="revolute">
-        <parent link="link1" />
-        <child link="link2" />
+        <parent link="Rlink1" />
+        <child link="Rlink2" />
         <origin xyz="0.0 0 0" rpy="0 0 0" />
         <limit lower="-2.53" upper="2.53" effort="10" velocity="3" />
@@ -304,6 +304,6 @@
         </joint>
         <joint name="Rarm2_joint" type="revolute">
-        <parent link="link2" />
-        <child link="link3" />
+        <parent link="Rlink2" />
+        <child link="Rlink3" />
         <origin xyz="0.0797 0 0" rpy="0 0 0" />
         <limit lower="-2.53" upper="2.53" effort="10" velocity="3" />
@@ -312,6 +312,6 @@
         </joint>
         <joint name="Rarm3_joint" type="revolute">
-        <parent link="link3" />
-        <child link="link4" />
+        <parent link="Rlink3" />
+        <child link="Rlink4" />
         <origin xyz="0.053 0 0" rpy="0 0 0" />
         <limit lower="-2.53" upper="2.53" effort="10" velocity="3" />
@@ -320,6 +320,6 @@
         </joint>
         <joint name="Rarm4_joint" type="revolute">
-        <parent link="link4" />
-        <child link="link5" />
+        <parent link="Rlink4" />
+        <child link="Rlink5" />
         <origin xyz="0.026 0 0" rpy="0 0 0" />
         <limit lower="-2.53" upper="2.53" effort="10" velocity="3" />
@@ -328,6 +328,6 @@
         </joint>
         <joint name="Rarm5_joint" type="revolute">
-        <parent link="link5" />
-        <child link="link6" />
+        <parent link="Rlink5" />
+        <child link="Rlink6" />
         <origin xyz="0.0675 0 0" rpy="0 0 0" />
         <limit lower="-2.53" upper="2.53" effort="10" velocity="3" />
@@ -347,5 +347,5 @@
         <parent link="Llink2" />
         <child link="Llink3" />
-        <origin xyz="0.052 0 0" rpy="0 0 0" />
+        <origin xyz="0.0797 0 0" rpy="0 0 0" />
         <limit lower="-2.53" upper="2.53" effort="10" velocity="3" />
         <axis xyz="0 1 0" />
@@ -355,5 +355,5 @@
         <parent link="Llink3" />
         <child link="Llink4" />
-        <origin xyz="0.0815 0 0" rpy="0 0 0" />
+        <origin xyz="0.053 0 0" rpy="0 0 0" />
         <limit lower="-2.53" upper="2.53" effort="10" velocity="3" />
         <axis xyz="1 0 0" />
@@ -363,5 +363,5 @@
         <parent link="Llink4" />
         <child link="Llink5" />
-        <origin xyz="0.0415 0 0" rpy="0 0 0" />
+        <origin xyz="0.026 0 0" rpy="0 0 0" />
         <limit lower="-2.53" upper="2.53" effort="10" velocity="3" />
         <axis xyz="0 1 0" />
@@ -371,5 +371,5 @@
         <parent link="Llink5" />
         <child link="Llink6" />
-        <origin xyz="0.052 0 0" rpy="0 0 0" />
+        <origin xyz="0.0675 0 0" rpy="0 0 0" />
         <limit lower="-2.53" upper="2.53" effort="10" velocity="3" />
         <axis xyz="0 1 0" />

Commit message: Start of Firefinder, motion control, etc...

File: eurobot2014/eurobot2014_models/urdf/test.urdf.xacro (robot description, xacro)
@@ -254,5 +254,5 @@
         <parent link="base_link" />
         <child link="arm_level_link" />
-        <origin xyz="0 0 0.147" rpy="0 0 0" />
+        <origin xyz="0 0 0.130" rpy="0 0 0" />
         </joint>
         <joint name="rightarm_joint" type="fixed">

Commit message: Some improvements in Pathplanner and Pathwrapper. (init phase)

File: eurobot2014/eurobot2014_models/urdf/test.urdf.xacro (robot description, xacro)
@@ -204,4 +204,10 @@
                 <xacro:ax12_color />
         </xacro:my_cylinder>
+        <xacro:my_cylinder name="gros_base_laser_link" l="0.002" r="0.05" xyz="0 0 0" rpy="0 0 0" mass="0.5" material="Gazebo/FlatBlack">
+                <xacro:ax12_color />
+        </xacro:my_cylinder>
+        <xacro:my_cylinder name="gros_neato_link" l="0.002" r="0.05" xyz="0 0 0" rpy="0 0 0" mass="0.5" material="Gazebo/FlatBlack">
+                <xacro:ax12_color />
+        </xacro:my_cylinder>
  	<!-- ============================   Arms   ============================ -->
                 <xacro:my_box name="Rlink1" lwh="0.04 0.04 0.04" xyz="-0.02 0 0" rpy="0 0 0" mass="0.055" material="Gazebo/FlatBlack">
@@ -294,4 +300,14 @@
         <origin xyz="0 0 -0.035" rpy="0 0 1.5707963267" />
         </joint>
+        <joint name="gros_base_laser_joint" type="fixed">
+        <parent link="top_level" />
+        <child link="gros_base_laser_link" />
+        <origin xyz="0.0 0.0 -0.04" rpy="0 0 0" />
+        </joint>
+        <joint name="gros_neato_joint" type="fixed">
+        <parent link="gros_base_laser_link" />
+        <child link="gros_neato_link" />
+        <origin xyz="0 0.0 0.0" rpy="3.141592653 0 0" />
+        </joint>
  	<!-- =================== RIGHT ARM Definitions ==================== -->
         <joint name="Rarm1_joint" type="revolute">

Commit message: Add two simple simulators. (ARM and little base)

File: eurobot2014/eurobot2014_models/urdf/test.urdf.xacro (robot description, xacro)
@@ -352,5 +352,5 @@
         </joint>
 	<!-- =================== LEFT ARM Definitions ==================== -->
-        <joint name="Ljoint1" type="revolute">
+        <joint name="Larm1_joint" type="revolute">
         <parent link="Llink1" />
         <child link="Llink2" />
@@ -360,5 +360,5 @@
         <dynamics damping="0.0"/>
         </joint>
-        <joint name="Ljoint2" type="revolute">
+        <joint name="Larm2_joint" type="revolute">
         <parent link="Llink2" />
         <child link="Llink3" />
@@ -368,5 +368,5 @@
         <dynamics damping="0.0"/>
         </joint>
-        <joint name="Ljoint3" type="revolute">
+        <joint name="Larm3_joint" type="revolute">
         <parent link="Llink3" />
         <child link="Llink4" />
@@ -376,5 +376,5 @@
         <dynamics damping="0.0"/>
         </joint>
-        <joint name="Ljoint4" type="revolute">
+        <joint name="Larm4_joint" type="revolute">
         <parent link="Llink4" />
         <child link="Llink5" />
@@ -384,5 +384,5 @@
         <dynamics damping="0.0"/>
         </joint>
-        <joint name="Ljoint5" type="revolute">
+        <joint name="Larm5_joint" type="revolute">
         <parent link="Llink5" />
         <child link="Llink6" />
