Commit message: Some moves with the arms. Change in kinematics. Cleaning some files.

File: eurobot2014/eurobot2014_models/urdf/test.urdf.xacro (robot description, xacro)
@@ -211,39 +211,75 @@
         </xacro:my_cylinder>
  	<!-- ============================   Arms   ============================ -->
-                <xacro:my_box name="Rlink1" lwh="0.04 0.04 0.04" xyz="-0.02 0 0" rpy="0 0 0" mass="0.055" material="Gazebo/FlatBlack">
-                        <xacro:ax12_color />
-                </xacro:my_box>
-		<xacro:my_box name="Rlink2" lwh="0.0797 0.04 0.04" xyz="0.03985 0 0" rpy="0 0 0" mass="0.055" material="Gazebo/WhiteEmissive">
-                        <xacro:bracket_color />
-                </xacro:my_box>
-                <xacro:my_box name="Rlink3" lwh="0.053 0.04 0.04" xyz="0.0265 0 0" rpy="0 0 0" mass="0.05" material="Gazebo/FlatBlack">
-                        <xacro:ax12_color />
-                </xacro:my_box>
-                <xacro:my_box name="Rlink4" lwh="0.026 0.04 0.04" xyz="0.013 0 0" rpy="0 0 0" mass="0.05" material="Gazebo/WhiteEmissive">
-                        <xacro:bracket_color />
-                </xacro:my_box>
-                <xacro:my_box name="Rlink5" lwh="0.0675 0.04 0.04" xyz="0.03375 0 0" rpy="0 0 0" mass="0.05" material="Gazebo/FlatBlack">
-                        <xacro:ax12_color />
-                </xacro:my_box>
-                <xacro:my_box name="Rlink6" lwh="0.04 0.04 0.04" xyz="0.02 0 0" rpy="0 0 0" mass="0.05" material="Gazebo/WhiteEmissive">
-                        <xacro:bracket_color />
-                </xacro:my_box>
-                <xacro:my_box name="Llink1" lwh="0.04 0.04 0.04" xyz="-0.02 0 0" rpy="0 0 0" mass="0.055" material="Gazebo/FlatBlack">
-                        <xacro:ax12_color />
-                </xacro:my_box>
-                <xacro:my_box name="Llink2" lwh="0.0797 0.04 0.04" xyz="0.03985 0 0" rpy="0 0 0" mass="0.055" material="Gazebo/WhiteEmissive">
-                        <xacro:bracket_color />
-                </xacro:my_box>
-                <xacro:my_box name="Llink3" lwh="0.053 0.04 0.04" xyz="0.0265 0 0" rpy="0 0 0" mass="0.05" material="Gazebo/FlatBlack">
-                        <xacro:ax12_color />
-                </xacro:my_box>
-                <xacro:my_box name="Llink4" lwh="0.026 0.04 0.04" xyz="0.013 0 0" rpy="0 0 0" mass="0.05" material="Gazebo/WhiteEmissive">
-                        <xacro:bracket_color />
-                </xacro:my_box>
-                <xacro:my_box name="Llink5" lwh="0.0675 0.04 0.04" xyz="0.03375 0 0" rpy="0 0 0" mass="0.05" material="Gazebo/FlatBlack">
-                        <xacro:ax12_color />
-                </xacro:my_box>
-                <xacro:my_box name="Llink6" lwh="0.04 0.04 0.04" xyz="0.02 0 0" rpy="0 0 0" mass="0.05" material="Gazebo/WhiteEmissive">
-                        <xacro:bracket_color />
+                <xacro:my_box name="Rlink1" lwh="0.04 0.048 0.04" xyz="-0.02 0 0" rpy="0 0 0" mass="0.055" material="Gazebo/FlatBlack">
+                        <xacro:ax12_color />
+                </xacro:my_box>
+		<xacro:my_box name="Rlink2" lwh="0.0797 0.048 0.04" xyz="0.03985 0 0" rpy="0 0 0" mass="0.055" material="Gazebo/WhiteEmissive">
+                        <xacro:bracket_color />
+                </xacro:my_box>
+                <xacro:my_box name="Rlink3" lwh="0.053 0.048 0.04" xyz="0.0265 0 0" rpy="0 0 0" mass="0.05" material="Gazebo/FlatBlack">
+                        <xacro:ax12_color />
+                </xacro:my_box>
+                <xacro:my_box name="Rlink4" lwh="0.052 0.048 0.04" xyz="0.026 0 0" rpy="0 0 0" mass="0.05" material="Gazebo/WhiteEmissive">
+                        <xacro:bracket_color />
+                </xacro:my_box>
+                <xacro:my_box name="Rlink5" lwh="0.0675 0.048 0.04" xyz="0.03375 0 0" rpy="0 0 0" mass="0.05" material="Gazebo/FlatBlack">
+                        <xacro:ax12_color />
+                </xacro:my_box>
+                <xacro:my_box name="Rlink6" lwh="0.0415 0.048 0.04" xyz="0.02075 0 0" rpy="0 0 0" mass="0.05" material="Gazebo/WhiteEmissive">
+                        <xacro:bracket_color />
+                </xacro:my_box>
+                <xacro:my_box name="Rlink7" lwh="0.0001 0.0001 0.0001" xyz="0.00005 0 0" rpy="0 0 0" mass="0.05" material="Gazebo/WhiteEmissive">
+                        <xacro:bracket_color />
+                </xacro:my_box>
+                <xacro:my_box name="Rlink_base_grip" lwh="0.04 0.061 0.04" xyz="0.0 0 0" rpy="0 0 0" mass="0.05" material="Gazebo/WhiteEmissive">
+                        <xacro:bracket_color />
+                </xacro:my_box>
+                <xacro:my_box name="Rlink_finger1" lwh="0.007 0.007 0.034" xyz="0.0 0 0" rpy="0 0 0" mass="0.05" material="Gazebo/FlatBlack">
+                        <xacro:ax12_color />
+                </xacro:my_box>
+                <xacro:my_box name="Rlink_finger2" lwh="0.007 0.007 0.034" xyz="0.0 0 0" rpy="0 0 0" mass="0.05" material="Gazebo/FlatBlack">
+                        <xacro:ax12_color />
+                </xacro:my_box>
+                <xacro:my_box name="Rlink_pump1" lwh="0.022 0.01 0.01" xyz="0.0 0 0" rpy="0 0 0" mass="0.05" material="Gazebo/FlatBlack">
+                        <xacro:ax12_color />
+                </xacro:my_box>
+                <xacro:my_box name="Rlink_pump2" lwh="0.022 0.01 0.01" xyz="0.0 0 0" rpy="0 0 0" mass="0.05" material="Gazebo/FlatBlack">
+                        <xacro:ax12_color />
+                </xacro:my_box>
+                <xacro:my_box name="Llink1" lwh="0.04 0.048 0.04" xyz="-0.02 0 0" rpy="0 0 0" mass="0.055" material="Gazebo/FlatBlack">
+                        <xacro:ax12_color />
+                </xacro:my_box>
+                <xacro:my_box name="Llink2" lwh="0.0797 0.048 0.04" xyz="0.03985 0 0" rpy="0 0 0" mass="0.055" material="Gazebo/WhiteEmissive">
+                        <xacro:bracket_color />
+                </xacro:my_box>
+                <xacro:my_box name="Llink3" lwh="0.053 0.048 0.04" xyz="0.0265 0 0" rpy="0 0 0" mass="0.05" material="Gazebo/FlatBlack">
+                        <xacro:ax12_color />
+                </xacro:my_box>
+                <xacro:my_box name="Llink4" lwh="0.052 0.048 0.04" xyz="0.026 0 0" rpy="0 0 0" mass="0.05" material="Gazebo/WhiteEmissive">
+                        <xacro:bracket_color />
+                </xacro:my_box>
+                <xacro:my_box name="Llink5" lwh="0.0675 0.048 0.04" xyz="0.03375 0 0" rpy="0 0 0" mass="0.05" material="Gazebo/FlatBlack">
+                        <xacro:ax12_color />
+                </xacro:my_box>
+                <xacro:my_box name="Llink6" lwh="0.04 0.048 0.04" xyz="0.02 0 0" rpy="0 0 0" mass="0.05" material="Gazebo/WhiteEmissive">
+                        <xacro:bracket_color />
+                </xacro:my_box>
+                <xacro:my_box name="Llink7" lwh="0.0001 0.0001 0.0001" xyz="0.00005 0 0" rpy="0 0 0" mass="0.05" material="Gazebo/WhiteEmissive">
+                        <xacro:bracket_color />
+                </xacro:my_box>
+                <xacro:my_box name="Llink_base_grip" lwh="0.04 0.061 0.04" xyz="0.0 0 0" rpy="0 0 0" mass="0.05" material="Gazebo/WhiteEmissive">
+                        <xacro:bracket_color />
+                </xacro:my_box>
+                <xacro:my_box name="Llink_finger1" lwh="0.007 0.007 0.034" xyz="0.0 0 0" rpy="0 0 0" mass="0.05" material="Gazebo/FlatBlack">
+                        <xacro:ax12_color />
+                </xacro:my_box>
+                <xacro:my_box name="Llink_finger2" lwh="0.007 0.007 0.034" xyz="0.0 0 0" rpy="0 0 0" mass="0.05" material="Gazebo/FlatBlack">
+                        <xacro:ax12_color />
+                </xacro:my_box>
+                <xacro:my_box name="Llink_pump1" lwh="0.022 0.01 0.01" xyz="0.0 0 0" rpy="0 0 0" mass="0.05" material="Gazebo/FlatBlack">
+                        <xacro:ax12_color />
+                </xacro:my_box>
+                <xacro:my_box name="Llink_pump2" lwh="0.022 0.01 0.01" xyz="0.0 0 0" rpy="0 0 0" mass="0.05" material="Gazebo/FlatBlack">
+                        <xacro:ax12_color />
                 </xacro:my_box>
 	<!-- =================== Joint Definitions ==================== -->
@@ -338,6 +374,6 @@
         <parent link="Rlink4" />
         <child link="Rlink5" />
-        <origin xyz="0.026 0 0" rpy="0 0 0" />
-        <limit lower="-1.57" upper="1.57" effort="10" velocity="3" />
+        <origin xyz="0.052 0 0" rpy="0 0 0" />
+        <limit lower="-2.3" upper="2.3" effort="10" velocity="3" />
         <axis xyz="0 1 0" />
         <dynamics damping="0.0"/>
@@ -351,4 +387,37 @@
         <dynamics damping="0.0"/>
         </joint>
+        <joint name="Rarm6_joint" type="revolute">
+        <parent link="Rlink6" />
+        <child link="Rlink7" />
+        <origin xyz="0.0 0 0" rpy="0 0 0" />
+        <limit lower="-2.53" upper="2.53" effort="10" velocity="3" />
+        <axis xyz="1 0 0" />
+        <dynamics damping="0.0"/>
+        </joint>
+        <joint name="Rlink_base_grip_joint" type="fixed">
+        <parent link="Rlink6" />
+        <child link="Rlink_base_grip" />
+        <origin xyz="0.023 0.0 0.039" rpy="0 0 0" />
+        </joint>
+        <joint name="Rlink_finger1_joint" type="fixed">
+        <parent link="Rlink_base_grip" />
+        <child link="Rlink_finger1" />
+        <origin xyz="0.0 0.027 0.037" rpy="0 0 0" />
+        </joint>
+        <joint name="Rlink_finger2_joint" type="fixed">
+        <parent link="Rlink_base_grip" />
+        <child link="Rlink_finger2" />
+        <origin xyz="0.0 -0.027 0.037" rpy="0 0 0" />
+        </joint>
+        <joint name="Rlink_pump1_joint" type="fixed">
+        <parent link="Rlink6" />
+        <child link="Rlink_pump1" />
+        <origin xyz="0.0525 0.015 0.0" rpy="0 0 0" />
+        </joint>
+        <joint name="Rlink_pump2_joint" type="fixed">
+        <parent link="Rlink6" />
+        <child link="Rlink_pump2" />
+        <origin xyz="0.0525 -0.015 0.0" rpy="0 0 0" />
+        </joint>
 	<!-- =================== LEFT ARM Definitions ==================== -->
         <joint name="Larm1_joint" type="revolute">
@@ -379,5 +448,5 @@
         <parent link="Llink4" />
         <child link="Llink5" />
-        <origin xyz="0.026 0 0" rpy="0 0 0" />
+        <origin xyz="0.052 0 0" rpy="0 0 0" />
         <limit lower="-2.53" upper="2.53" effort="10" velocity="3" />
         <axis xyz="0 1 0" />
@@ -392,4 +461,37 @@
         <dynamics damping="0.0"/>
         </joint>
+        <joint name="Larm6_joint" type="revolute">
+        <parent link="Llink6" />
+        <child link="Llink7" />
+        <origin xyz="0.0 0 0" rpy="0 0 0" />
+        <limit lower="-2.53" upper="2.53" effort="10" velocity="3" />
+        <axis xyz="1 0 0" />
+        <dynamics damping="0.0"/>
+        </joint>
+        <joint name="Llink_base_grip_joint" type="fixed">
+        <parent link="Llink6" />
+        <child link="Llink_base_grip" />
+        <origin xyz="0.023 0.0 0.039" rpy="0 0 0" />
+        </joint>
+        <joint name="Llink_finger1_joint" type="fixed">
+        <parent link="Llink_base_grip" />
+        <child link="Llink_finger1" />
+        <origin xyz="0.0 0.027 0.037" rpy="0 0 0" />
+        </joint>
+        <joint name="Llink_finger2_joint" type="fixed">
+        <parent link="Llink_base_grip" />
+        <child link="Llink_finger2" />
+        <origin xyz="0.0 -0.027 0.037" rpy="0 0 0" />
+        </joint>
+        <joint name="Llink_pump1_joint" type="fixed">
+        <parent link="Llink6" />
+        <child link="Llink_pump1" />
+        <origin xyz="0.0525 0.015 0.0" rpy="0 0 0" />
+        </joint>
+        <joint name="Llink_pump2_joint" type="fixed">
+        <parent link="Llink6" />
+        <child link="Llink_pump2" />
+        <origin xyz="0.0525 -0.015 0.0" rpy="0 0 0" />
+        </joint>
 	<gazebo reference="indomptable">
   	</gazebo>

Commit message: First odometry calibration for GROS.

File: eurobot2014/eurobot2014_models/urdf/test.urdf.xacro (robot description, xacro)
@@ -296,15 +296,15 @@
         <parent link="base_link" />
         <child link="arm_level_link" />
-        <origin xyz="0 0 0.130" rpy="0 0 0" />
+        <origin xyz="0 0 0.180" rpy="0 0 0" />
         </joint>
         <joint name="rightarm_joint" type="fixed">
         <parent link="arm_level_link" />
         <child link="Rlink1" />
-        <origin xyz="0.05 -0.06 0.032" rpy="0 0 0" />
+        <origin xyz="0.05 -0.075 0.032" rpy="0 0 0" />
         </joint>
         <joint name="leftarm_joint" type="fixed">
         <parent link="arm_level_link" />
         <child link="Llink1" />
-        <origin xyz="0.05 0.06 0.032" rpy="0 0 0" />
+        <origin xyz="0.05 0.075 0.032" rpy="0 0 0" />
         </joint>
         <joint name="left_panel_joint" type="fixed">

Commit message: Navigation stack for GROS.

File: eurobot2014/eurobot2014_models/urdf/test.urdf.xacro (robot description, xacro)
@@ -324,15 +324,16 @@
         </joint>
 	<!-- =================== LASER Definitions ==================== -->
-        <joint name="base_laser_joint" type="prismatic">
+        <!--<joint name="base_laser_joint" type="prismatic">-->
+	<joint name="base_laser_joint" type="fixed">
         <parent link="base_link" />
         <child link="base_laser" />
         <origin xyz="0.15 0 0.07" rpy="0 0 0" />
-        <limit lower="0.0" upper="0.1" effort="10" velocity="3" />
-        <axis xyz="0 0 1" />
+        <!--<limit lower="0.0" upper="0.1" effort="10" velocity="3" />
+        <axis xyz="0 0 1" />-->
         </joint>
         <joint name="laser_joint" type="fixed">
         <parent link="base_laser" />
         <child link="hokuyo_laser" />
-        <origin xyz="0 0 -0.035" rpy="0 0 1.5707963267" />
+        <origin xyz="0 0 -0.035" rpy="3.141592653 0 0" />
         </joint>
         <joint name="gros_base_laser_joint" type="fixed">

Commit message: Add a new AX12 to move the laser.

File: eurobot2014/eurobot2014_models/urdf/test.urdf.xacro (robot description, xacro)
@@ -324,11 +324,11 @@
         </joint>
 	<!-- =================== LASER Definitions ==================== -->
-        <!--<joint name="base_laser_joint" type="prismatic">-->
-	<joint name="base_laser_joint" type="fixed">
+        <joint name="base_laser_joint" type="prismatic">
+	<!--<joint name="base_laser_joint" type="fixed">-->
         <parent link="base_link" />
         <child link="base_laser" />
         <origin xyz="0.15 0 0.07" rpy="0 0 0" />
-        <!--<limit lower="0.0" upper="0.1" effort="10" velocity="3" />
-        <axis xyz="0 0 1" />-->
+        <limit lower="0.0" upper="0.15" effort="10" velocity="3" />
+        <axis xyz="0 0 1" />
         </joint>
         <joint name="laser_joint" type="fixed">
