Commit message: Some saving. Not important stuff.

File: nestor/nestor_model/urdf/nestor.urdf.xacro (robot description, xacro)
@@ -204,4 +204,10 @@
 		<xacro:grey2 />
 	</xacro:my_cylinder>
+        <xacro:my_box name="base_laser" lwh="0.05 0.05 0.041" xyz="0 0 0" rpy="0 0 0" mass="0.5" material="Gazebo/FlatBlack">
+                <xacro:ax12_color />
+        </xacro:my_box>
+        <xacro:my_cylinder name="hokuyo_laser" l="0.029" r="0.021" xyz="0 0 0" rpy="0 0 0" mass="0.5" material="Gazebo/FlatBlack">
+                <xacro:ax12_color />
+        </xacro:my_cylinder>
 	<xacro:my_box name="level1_link" lwh="0.25 0.34 0.002" xyz="0 0 0" rpy="0 0 0" mass="0.1" material="Gazebo/Grey">
 		<xacro:grey2 />
@@ -264,4 +270,5 @@
  	-->
  	<!-- ============================   Arms   ============================ -->
+<!--
                 <xacro:my_box name="shoulder_yaw_link" lwh="0.05 0.05 0.05" xyz="0.0 0.0 0.0" rpy="0 0 0" mass="0.055" material="Gazebo/WhiteEmissive">
                         <xacro:bracket_color />
@@ -285,4 +292,5 @@
                         <xacro:ax12_color />
                 </xacro:my_box>
+-->
 <!--
 	<xacro:macro name="arm" params="side reflect">
@@ -356,4 +364,15 @@
         <axis xyz="1 0 0" />
         </joint>
+        <joint name="base_laser_joint" type="fixed">
+        <parent link="plate_link" />
+        <child link="base_laser" />
+        <origin xyz="0.05 0 -0.021" rpy="0 0 0" />
+        <axis xyz="0 0 1" />
+        </joint>
+        <joint name="laser_joint" type="fixed">
+        <parent link="base_laser" />
+        <child link="hokuyo_laser" />
+        <origin xyz="0 0 -0.035" rpy="3.141592653 0 0" />
+        </joint>
         <joint name="level1_joint" type="fixed">
         <parent link="base_link" />
@@ -416,4 +435,5 @@
         <axis xyz="1 0 0" />
         </joint>
+<!--
         <joint name="shoulder_yaw_joint" type="revolute">
         <parent link="level2_link" />
@@ -470,4 +490,5 @@
         <dynamics damping="0.0"/>
         </joint>
+-->
 <!-- Finger joint -->
 	<!--

Commit message: [NESTOR] Update urdf for robot ARM.

File: nestor/nestor_model/urdf/nestor.urdf.xacro (robot description, xacro)
@@ -240,4 +240,26 @@
 		<xacro:grey2 />
 	</xacro:my_cylinder>
+ 	<!-- ============================   Arms   ============================ -->
+	<xacro:my_box name="arm_base_link" lwh="0.05 0.05 0.05" xyz="0.0 0.0 0.0" rpy="0 0 0" mass="0.055" material="Gazebo/WhiteEmissive">
+		<xacro:bracket_color />
+	</xacro:my_box>
+	<xacro:my_box name="shoulder_yaw_link" lwh="0.05 0.05 0.05" xyz="0.0 0.0 0.0" rpy="0 0 0" mass="0.055" material="Gazebo/WhiteEmissive">
+		<xacro:bracket_color />
+	</xacro:my_box>
+	<xacro:my_box name="shoulder_pitch_link" lwh="0.05 0.05 0.05" xyz="0.0 0.0 0.0" rpy="0 0 0" mass="0.055" material="Gazebo/WhiteEmissive">
+		<xacro:bracket_color />
+	</xacro:my_box>
+	<xacro:my_box name="elbow_pitch_link" lwh="0.05 0.05 0.05" xyz="0.0 0.0 0.0" rpy="0 0 0" mass="0.055" material="Gazebo/WhiteEmissive">
+		<xacro:bracket_color />
+	</xacro:my_box>
+	<xacro:my_box name="wrist_pitch_link" lwh="0.05 0.05 0.05" xyz="0.0 0.0 0.0" rpy="0 0 0" mass="0.055" material="Gazebo/WhiteEmissive">
+		<xacro:bracket_color />
+	</xacro:my_box>
+	<xacro:my_box name="wrist_yaw_link" lwh="0.05 0.05 0.05" xyz="0.0 0.0 0.0" rpy="0 0 0" mass="0.055" material="Gazebo/WhiteEmissive">
+		<xacro:bracket_color />
+	</xacro:my_box>
+	<xacro:my_box name="wrist_roll_link" lwh="0.05 0.05 0.05" xyz="0.0 0.0 0.0" rpy="0 0 0" mass="0.055" material="Gazebo/WhiteEmissive">
+		<xacro:bracket_color />
+	</xacro:my_box>
  	<!--
 	<xacro:my_box name="base_laser_bottom" lwh="0.05 0.05 0.041" xyz="0 0 0" rpy="0 0 0" mass="0.1" material="Gazebo/FlatBlack">
@@ -435,10 +457,16 @@
         <axis xyz="1 0 0" />
         </joint>
-<!--
+	<!-- ARM -->
+	<joint name="arm_base_joint" type="fixed">
+        <parent link="level1_link" />
+        <child link="arm_base_link" />
+        <origin xyz="0.065 0.0 0.165" rpy="0 0 0" />
+        <axis xyz="1 0 0" />
+        </joint>
         <joint name="shoulder_yaw_joint" type="revolute">
-        <parent link="level2_link" />
+        <parent link="arm_base_link" />
         <child link="shoulder_yaw_link" />
-        <origin xyz="0.085 0.0 0.025" rpy="0 0 0" />
-        <limit lower="-1.57" upper="1.57" effort="10" velocity="3" />
+        <origin xyz="0.0 0.0 0.0" rpy="0 0 0" />
+        <limit lower="-1.3" upper="1.3" effort="10" velocity="3" />
         <axis xyz="0 0 1" />
         <dynamics damping="0.0"/>
@@ -447,6 +475,6 @@
         <parent link="shoulder_yaw_link" />
         <child link="shoulder_pitch_link" />
-        <origin xyz="0.0 0.0 0.08" rpy="0 0 0" />
-        <limit lower="-0.625" upper="0.625" effort="10" velocity="3" />
+        <origin xyz="0.0 0.0 0.0" rpy="0 0 0" />
+        <limit lower="-0.5" upper="1.4" effort="10" velocity="3" />
         <axis xyz="0 1 0" />
         <dynamics damping="0.0"/>
@@ -455,40 +483,32 @@
         <parent link="shoulder_pitch_link" />
         <child link="elbow_pitch_link" />
-        <origin xyz="0.4 0.0 0" rpy="0 0 0" />
-        <limit lower="-2.53" upper="2.53" effort="10" velocity="3" />
-        <axis xyz="0 1 0" />
-        <dynamics damping="0.0"/>
-        </joint>
-        <joint name="wrist_fixed_joint" type="fixed">
+        <origin xyz="0.3 0.0 0" rpy="0 0 0" />
+        <limit lower="-1.57" upper="1.57" effort="10" velocity="3" />
+        <axis xyz="0 1 0" />
+        <dynamics damping="0.0"/>
+        </joint>
+        <joint name="wrist_pitch_joint" type="fixed">
         <parent link="elbow_pitch_link" />
         <child link="wrist_pitch_link" />
-        <origin xyz="0.3 -0.04 0.0" rpy="0 0 0" />
-        <axis xyz="1 0 0" />
-        </joint>
-        <joint name="wrist_pitch_joint" type="revolute">
+        <origin xyz="0.2 0.0 0.0" rpy="0 0 0" />
+        <limit lower="-1.57" upper="1.57" effort="10" velocity="3" />
+        <axis xyz="0 1 0" />
+        </joint>
+        <joint name="wrist_yaw_joint" type="revolute">
         <parent link="wrist_pitch_link" />
         <child link="wrist_yaw_link" />
-        <origin xyz="0.0 0.04 0" rpy="0 0 0" />
-        <limit lower="-2.53" upper="2.53" effort="10" velocity="3" />
-        <axis xyz="0 1 0" />
-        <dynamics damping="0.0"/>
-        </joint>
-        <joint name="wrist_yaw_joint" type="revolute">
+        <origin xyz="0.05 0.0 0" rpy="0 0 0" />
+        <limit lower="-1.53" upper="1.53" effort="10" velocity="3" />
+        <axis xyz="0 0 1" />
+        <dynamics damping="0.0"/>
+        </joint>
+        <joint name="wrist_roll_joint" type="revolute">
         <parent link="wrist_yaw_link" />
         <child link="wrist_roll_link" />
-        <origin xyz="0.0 0.0 -0.065" rpy="0 0 0" />
-        <limit lower="-2.53" upper="2.53" effort="10" velocity="3" />
-        <axis xyz="0 0 1" />
-        <dynamics damping="0.0"/>
-        </joint>
-        <joint name="wrist_roll_joint" type="revolute">
-        <parent link="wrist_roll_link" />
-        <child link="claw_link" />
-        <origin xyz="0.08 0.0 0.0" rpy="0 0 0" />
-        <limit lower="-2.53" upper="2.53" effort="10" velocity="3" />
-        <axis xyz="1 0 0" />
-        <dynamics damping="0.0"/>
-        </joint>
--->
+        <origin xyz="0.05 0.0 0.0" rpy="0 0 0" />
+        <limit lower="-1.53" upper="1.53" effort="10" velocity="3" />
+        <axis xyz="1 0 0" />
+        <dynamics damping="0.0"/>
+        </joint>
 <!-- Finger joint -->
 	<!--

Commit message: [NESTOR] Update urdf for robot ARM.

File: nestor/nestor_model/urdf/nestor.urdf.xacro (robot description, xacro)
@@ -5,5 +5,5 @@
        xmlns:interface="http://playerstage.sourceforge.net/gazebo/xmlschema/#interface"
        xmlns:xacro="http://ros.org/wiki/xacro"
-	   name="indomptable">
+	   name="NESTOR">
 	<!--
 	<include filename="$(find pi_robot_description)/urdf/sensors/hokuyo_laser_gazebo.xacro" />
@@ -488,5 +488,5 @@
         <dynamics damping="0.0"/>
         </joint>
-        <joint name="wrist_pitch_joint" type="fixed">
+        <joint name="wrist_pitch_joint" type="revolute">
         <parent link="elbow_pitch_link" />
         <child link="wrist_pitch_link" />
@@ -872,5 +872,5 @@
 	</joint>
 	-->
-	<gazebo reference="indomptable">
+	<gazebo reference="NESTOR">
   	</gazebo>
 </robot>

Commit message: [NESTOR] Add amcl launch file.

File: nestor/nestor_model/urdf/nestor.urdf.xacro (robot description, xacro)
@@ -231,11 +231,11 @@
 		<xacro:grey2 />
 	</xacro:my_box>
-	<xacro:my_cylinder name="head_tube1_link" l="0.650" r="0.006" xyz="0 0 0" rpy="0 0 0" mass="0.1" material="Gazebo/Grey">
-		<xacro:grey2 />
-	</xacro:my_cylinder>
-	<xacro:my_cylinder name="head_tube2_link" l="0.650" r="0.006" xyz="0 0 0" rpy="0 0 0" mass="0.1" material="Gazebo/Grey">
-		<xacro:grey2 />
-	</xacro:my_cylinder>
-	<xacro:my_cylinder name="head_tube3_link" l="0.650" r="0.006" xyz="0 0 0" rpy="0 0 0" mass="0.1" material="Gazebo/Grey">
+	<xacro:my_cylinder name="head_tube1_link" l="0.456" r="0.006" xyz="0 0 0" rpy="0 0 0" mass="0.1" material="Gazebo/Grey">
+		<xacro:grey2 />
+	</xacro:my_cylinder>
+	<xacro:my_cylinder name="head_tube2_link" l="0.456" r="0.006" xyz="0 0 0" rpy="0 0 0" mass="0.1" material="Gazebo/Grey">
+		<xacro:grey2 />
+	</xacro:my_cylinder>
+	<xacro:my_cylinder name="head_tube3_link" l="0.456" r="0.006" xyz="0 0 0" rpy="0 0 0" mass="0.1" material="Gazebo/Grey">
 		<xacro:grey2 />
 	</xacro:my_cylinder>
@@ -430,5 +430,5 @@
         <parent link="level1_link" />
         <child link="level2_link" />
-        <origin xyz="0.0 0.0 0.1" rpy="0 0 0" />
+        <origin xyz="0.0 0.0 0.301" rpy="0 0 0" />
         <axis xyz="1 0 0" />
         </joint>
@@ -436,5 +436,5 @@
         <parent link="level2_link" />
         <child link="head_base_link" />
-        <origin xyz="0.0 0.0 0.65" rpy="0 0 0" />
+        <origin xyz="0.0 0.0 0.456" rpy="0 0 0" />
         <axis xyz="1 0 0" />
         </joint>
@@ -442,5 +442,5 @@
         <parent link="level2_link" />
         <child link="head_tube1_link" />
-        <origin xyz="0.035 0.125 0.326" rpy="0 0 0" />
+        <origin xyz="0.035 0.125 0.228" rpy="0 0 0" />
         <axis xyz="1 0 0" />
         </joint>
@@ -448,5 +448,5 @@
         <parent link="level2_link" />
         <child link="head_tube2_link" />
-        <origin xyz="0.035 -0.125 0.326" rpy="0 0 0" />
+        <origin xyz="0.035 -0.125 0.228" rpy="0 0 0" />
         <axis xyz="1 0 0" />
         </joint>
@@ -454,5 +454,5 @@
         <parent link="level2_link" />
         <child link="head_tube3_link" />
-        <origin xyz="-0.065 0.0 0.326" rpy="0 0 0" />
+        <origin xyz="-0.065 0.0 0.228" rpy="0 0 0" />
         <axis xyz="1 0 0" />
         </joint>
@@ -476,5 +476,5 @@
         <child link="shoulder_pitch_link" />
         <origin xyz="0.0 0.0 0.0" rpy="0 0 0" />
-        <limit lower="-0.5" upper="1.4" effort="10" velocity="3" />
+        <limit lower="-1.5" upper="0.5" effort="10" velocity="3" />
         <axis xyz="0 1 0" />
         <dynamics damping="0.0"/>
@@ -484,5 +484,5 @@
         <child link="elbow_pitch_link" />
         <origin xyz="0.3 0.0 0" rpy="0 0 0" />
-        <limit lower="-1.57" upper="1.57" effort="10" velocity="3" />
+        <limit lower="-2.0" upper="2.0" effort="10" velocity="3" />
         <axis xyz="0 1 0" />
         <dynamics damping="0.0"/>
@@ -492,5 +492,5 @@
         <child link="wrist_pitch_link" />
         <origin xyz="0.2 0.0 0.0" rpy="0 0 0" />
-        <limit lower="-1.57" upper="1.57" effort="10" velocity="3" />
+        <limit lower="-2.0" upper="2.0" effort="10" velocity="3" />
         <axis xyz="0 1 0" />
         </joint>
@@ -499,5 +499,5 @@
         <child link="wrist_yaw_link" />
         <origin xyz="0.05 0.0 0" rpy="0 0 0" />
-        <limit lower="-1.53" upper="1.53" effort="10" velocity="3" />
+        <limit lower="-2.0" upper="2.0" effort="10" velocity="3" />
         <axis xyz="0 0 1" />
         <dynamics damping="0.0"/>
@@ -507,5 +507,5 @@
         <child link="wrist_roll_link" />
         <origin xyz="0.05 0.0 0.0" rpy="0 0 0" />
-        <limit lower="-1.53" upper="1.53" effort="10" velocity="3" />
+        <limit lower="-2.0" upper="2.0" effort="10" velocity="3" />
         <axis xyz="1 0 0" />
         <dynamics damping="0.0"/>

Commit message: [NESTOR] Add the global map.

File: nestor/nestor_model/urdf/nestor.urdf.xacro (robot description, xacro)
@@ -240,4 +240,7 @@
 		<xacro:grey2 />
 	</xacro:my_cylinder>
+	<xacro:my_box name="head_kinect_link" lwh="0.05 0.05 0.05" xyz="0 0 0" rpy="0 0 0" mass="0.1" material="Gazebo/Grey">
+                <xacro:grey2 />
+        </xacro:my_box>
  	<!-- ============================   Arms   ============================ -->
 	<xacro:my_box name="arm_base_link" lwh="0.05 0.05 0.05" xyz="0.0 0.0 0.0" rpy="0 0 0" mass="0.055" material="Gazebo/WhiteEmissive">
@@ -457,4 +460,10 @@
         <axis xyz="1 0 0" />
         </joint>
+	<joint name="head_kinect_joint" type="fixed">
+        <parent link="head_base_link" />
+        <child link="head_kinect_link" />
+        <origin xyz="0.0 0.0 0.06" rpy="0 0 0" />
+        <axis xyz="1 0 0" />
+        </joint>
 	<!-- ARM -->
 	<joint name="arm_base_joint" type="fixed">
